File: PathPal-PCB.kicad_sch (KiCad schematic)
At the start: 34 parts, among them J1 Raspberry_Pi_2_3, J2 Motor, J3 Button1, J4 Button2, J5 Button3, Q1 AO3400A, Q2 AO3400A, Q3 AO3400A, Q4 AO3400A, U1 Gyro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

Commit message: parts layout done
Parts:
- J3, J4, J5: footprint Connector_PinSocket_2.54mm:PinSocket_1x02_P2.54mm_Horizontal -> Connector_PinSocket_2.54mm:PinSocket_1x02_P2.54mm_Vertical
- U1: footprint Connector_PinSocket_2.54mm:PinSocket_1x08_P2.54mm_Horizontal -> Connector_PinSocket_2.54mm:PinSocket_1x08_P2.54mm_Vertical
- U2: footprint Connector_PinSocket_2.54mm:PinSocket_1x04_P2.54mm_Horizontal -> Connector_PinSocket_2.54mm:PinSocket_1x04_P2.54mm_Vertical
Changed lines of the file:
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@@
 			)
 		)
-		(property "Footprint" "Connector_PinSocket_2.54mm:PinSocket_1x04_P2.54mm_Horizontal"
+		(property "Footprint" "Connector_PinSocket_2.54mm:PinSocket_1x04_P2.54mm_Vertical"
 			(at 74.93 158.75 0)
 			(effects
@@
 			)
 		)
-		(property "Footprint" "Connector_PinSocket_2.54mm:PinSocket_1x02_P2.54mm_Horizontal"
+		(property "Footprint" "Connector_PinSocket_2.54mm:PinSocket_1x02_P2.54mm_Vertical"
 			(at 262.89 133.35 0)
 			(effects
@@
 			)
 		)
-		(property "Footprint" "Connector_PinSocket_2.54mm:PinSocket_1x02_P2.54mm_Horizontal"
+		(property "Footprint" "Connector_PinSocket_2.54mm:PinSocket_1x02_P2.54mm_Vertical"
 			(at 186.69 133.35 0)
 			(effects
@@
 			)
 		)
-		(property "Footprint" "Connector_PinSocket_2.54mm:PinSocket_1x08_P2.54mm_Horizontal"
+		(property "Footprint" "Connector_PinSocket_2.54mm:PinSocket_1x08_P2.54mm_Vertical"
 			(at 43.18 158.75 0)
 			(effects
@@
 			)
 		)
-		(property "Footprint" "Connector_PinSocket_2.54mm:PinSocket_1x02_P2.54mm_Horizontal"
+		(property "Footprint" "Connector_PinSocket_2.54mm:PinSocket_1x02_P2.54mm_Vertical"
 			(at 222.25 133.35 0)
 			(effects

Commit message: Fixed Routing
Parts:
- added J6: Motor, Connector_PinSocket_2.54mm:PinSocket_1x02_P2.54mm_Vertical, symbol Connector:Conn_01x02_Socket
- D2, D3: footprint LED_THT:LED_D5.0mm-4_RGB -> LED_THT:LED_D5.0mm-4_RGB_Wide_Pins
Connections:
- net GND: now also J6.2 (NEG-)
- net BatLow: now reaches J1.40 (GPIO21/SCLK1)
- net BatLow: now also J6.1 (POS+)
- no-connect marks 19 -> 18
Changed lines of the file:
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@@
 	)
 	(no_connect
-		(at 100.33 78.74)
-	)
-	(no_connect
 		(at 140.97 76.2)
 	)
@@
 	(wire
 		(pts
+			(xy 86.36 78.74) (xy 100.33 78.74)
+		)
+		(stroke
+			(width 0)
+			(type default)
+		)
+	)
+	(wire
+		(pts
 			(xy 248.92 133.35) (xy 248.92 138.43)
 		)
@@
 	(wire
 		(pts
+			(xy 50.8 77.47) (xy 50.8 80.01)
+		)
+		(stroke
+			(width 0)
+			(type default)
+		)
+	)
+	(wire
+		(pts
 			(xy 194.31 43.18) (xy 198.12 43.18)
 		)
@@
 	(wire
 		(pts
+			(xy 50.8 74.93) (xy 59.69 74.93)
+		)
+		(stroke
+			(width 0)
+			(type default)
+		)
+	)
+	(wire
+		(pts
 			(xy 177.8 100.33) (xy 186.69 100.33)
 		)
@@
 	(wire
 		(pts
+			(xy 50.8 77.47) (xy 59.69 77.47)
+		)
+		(stroke
+			(width 0)
+			(type default)
+		)
+	)
+	(wire
+		(pts
 			(xy 125.73 43.18) (xy 125.73 45.72)
 		)
@@
 		)
 	)
+	(label "BatLow"
+		(at 50.8 74.93 0)
+		(effects
+			(font
+				(size 1.27 1.27)
+			)
+			(justify left bottom)
+		)
+	)
 	(label "SCL"
 		(at 143.51 66.04 0)
@@
 		)
 	)
+	(label "BatLow"
+		(at 86.36 78.74 0)
+		(effects
+			(font
+				(size 1.27 1.27)
+			)
+			(justify left bottom)
+		)
+	)
 	(symbol
 		(lib_id "power:GND")
@@
 			)
 		)
-		(property "Footprint" "LED_THT:LED_D5.0mm-4_RGB"
+		(property "Footprint" "LED_THT:LED_D5.0mm-4_RGB_Wide_Pins"
 			(at 245.11 38.1 0)
 			(effects
@@
 	)
 	(symbol
+		(lib_id "power:GND")
+		(at 50.8 80.01 0)
+		(unit 1)
+		(exclude_from_sim no)
+		(in_bom yes)
+		(on_board yes)
+		(dnp no)
+		(fields_autoplaced yes)
+		(property "Reference" "#PWR024"
+			(at 50.8 86.36 0)
+			(effects
+				(font
+					(size 1.27 1.27)
+				)
+				(hide yes)
+			)
+		)
+		(property "Value" "GND"
+			(at 50.8 85.09 0)
+			(effects
+				(font
+					(size 1.27 1.27)
+				)
+			)
+		)
+		(property "Footprint" ""
+			(at 50.8 80.01 0)
+			(effects
+				(font
+					(size 1.27 1.27)
+				)
+				(hide yes)
+			)
+		)
+		(property "Datasheet" ""
+			(at 50.8 80.01 0)
+			(effects
+				(font
+					(size 1.27 1.27)
+				)
+				(hide yes)
+			)
+		)
+		(property "Description" "Power symbol creates a global label with name \"GND\" , ground"
+			(at 50.8 80.01 0)
+			(effects
+				(font
+					(size 1.27 1.27)
+				)
+				(hide yes)
+			)
+		)
+		(pin "1"
+		)
+		(instances
+			(project ""
+				(path "/5d170015-070c-4f9e-a723-d3289cd8d8fb"
+					(reference "#PWR024")
+					(unit 1)
+				)
+			)
+		)
+	)
+	(symbol
 		(lib_id "Device:LED_RGAB")
 		(at 245.11 62.23 0)
@@
 			)
 		)
-		(property "Footprint" "LED_THT:LED_D5.0mm-4_RGB"
+		(property "Footprint" "LED_THT:LED_D5.0mm-4_RGB_Wide_Pins"
 			(at 245.11 63.5 0)
 			(effects
@@
 					(unit 1)
 				)
+			)
+		)
+	)
+	(symbol
+		(lib_id "Connector:Conn_01x02_Socket")
+		(at 64.77 74.93 0)
+		(unit 1)
+		(exclude_from_sim no)
+		(in_bom yes)
+		(on_board yes)
+		(dnp no)
+		(property "Reference" "J6"
+			(at 60.198 71.374 0)
+			(effects
+				(font
+					(size 1.27 1.27)
+				)
+				(justify left)
+			)
+		)
+		(property "Value" "Motor"
+			(at 62.992 71.374 0)
+			(effects
+				(font
+					(size 1.27 1.27)
+				)
+				(justify left)
+			)
+		)
+		(property "Footprint" "Connector_PinSocket_2.54mm:PinSocket_1x02_P2.54mm_Vertical"
+			(at 64.77 74.93 0)
+			(effects
+				(font
+					(size 1.27 1.27)
+				)
+				(hide yes)
+			)
+		)
+		(property "Datasheet" "~"
+			(at 64.77 74.93 0)
+			(effects
+				(font
+					(size 1.27 1.27)
+				)
+				(hide yes)
+			)
+		)
+		(property "Description" "Generic connector, single row, 01x02, script generated"
+			(at 64.77 74.93 0)
+			(effects
+				(font
+					(size 1.27 1.27)
+				)
+				(hide yes)
+			)
+		)
+		(pin "2"
+		)
+		(pin "1"
+		)
+		(instances
+			(project "PathPal-PCB"
+				(path "/5d170015-070c-4f9e-a723-d3289cd8d8fb"
+					(reference "J6")
+					(unit 1)
+				)

Commit message: Order
Parts:
- U3: footprint Connector_JST:JST_GH_BM06B-GHS-TBT_1x06-1MP_P1.25mm_Vertical -> Connector_PinSocket_2.54mm:PinSocket_1x06_P2.54mm_Vertical
Changed lines of the file:
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@@
 		(title "PathPal PCB")
 		(date "2026-02-18")
-		(rev "V1")
+		(rev "V2")
 		(company "Senseway")
 	)
@@
 			)
 		)
-		(property "Footprint" "Connector_JST:JST_GH_BM06B-GHS-TBT_1x06-1MP_P1.25mm_Vertical"
+		(property "Footprint" "Connector_PinSocket_2.54mm:PinSocket_1x06_P2.54mm_Vertical"
 			(at 105.41 156.21 0)
 			(effects

Commit message: simpler
Parts:
- removed C1: 10uF, PCM_JLCPCB:C_0805, symbol PCM_JLCPCB-Capacitors:0805,10uF
- removed C2, C3, C4: 100nF, PCM_JLCPCB:C_0805, symbol PCM_JLCPCB-Capacitors:0805,100nF
- removed D1: 1N4148W, Diode_SMD:D_SOD-123, symbol Diode:1N4148W
- removed D2, D3: LED_RGAB, LED_THT:LED_D5.0mm-4_RGB_Wide_Pins, symbol Device:LED_RGAB
- removed J2, J6: Motor, Connector_PinSocket_2.54mm:PinSocket_1x02_P2.54mm_Vertical, symbol Connector:Conn_01x02_Socket
- removed J3: Button1, Connector_PinSocket_2.54mm:PinSocket_1x02_P2.54mm_Vertical, symbol Connector:Conn_01x02_Socket
- removed J4: Button2, Connector_PinSocket_2.54mm:PinSocket_1x02_P2.54mm_Vertical, symbol Connector:Conn_01x02_Socket
- removed J5: Button3, Connector_PinSocket_2.54mm:PinSocket_1x02_P2.54mm_Vertical, symbol Connector:Conn_01x02_Socket
- removed Q1, Q2, Q3, Q4: AO3400A, PCM_JLCPCB:Q_SOT-23, symbol PCM_JLCPCB-Transistors:NMOS,AO3400A
- removed R10, R15, R9: 10kΩ, PCM_JLCPCB:R_0805, symbol PCM_JLCPCB-Resistors:0805,10kΩ
- removed R11, R12, R13, R14: 100Ω, PCM_JLCPCB:R_0805, symbol PCM_JLCPCB-Resistors:0805,100Ω
- removed R3, R4, R5, R6: 1kΩ, PCM_JLCPCB:R_0805, symbol PCM_JLCPCB-Resistors:0805,1kΩ
- removed R7, R8: 150Ω, PCM_JLCPCB:R_0805, symbol PCM_JLCPCB-Resistors:0805,150Ω
- R1, R2: footprint PCM_JLCPCB:R_0805 -> Resistor_THT:R_Axial_DIN0207_L6.3mm_D2.5mm_P7.62mm_Horizontal
Connections:
- net BLedSEL: no longer names the net of J1.12 (GPIO18/PWM0)
- net BatLow: no longer names the net of J1.40 (GPIO21/SCLK1)
- net Button1IN: no longer names the net of J1.16 (GPIO23)
- net Button2IN: no longer names the net of J1.18 (GPIO24)
- net Button3IN: no longer names the net of J1.22 (GPIO25)
- net GLedSEL: no longer names the net of J1.33 (PWM1/GPIO13)
- net MotorSEL: no longer names the net of J1.11 (GPIO17)
- net RLedSEL: no longer names the net of J1.32 (PWM0/GPIO12)
- no-connect marks 18 -> 26
